Commit message: Albatross model added

File: urdf/quadrotor_base.urdf.xacro (robot description, xacro)
@@ -7,5 +7,5 @@
   <!-- Main quadrotor link -->
   <xacro:macro name="quadrotor_base_macro">
-    <link name="base_link">
+<!--    <link name="base_link">
       <inertial>
         <mass value="1.477" />
@@ -26,4 +26,45 @@
       </collision>
     </link>
+-->
+  <link
+    name="base_combined">
+    <inertial>
+      <origin
+        xyz="-0.000692090305311921 0.198982523237643 -0.0693208796289051"
+        rpy="0 0 0" />
+      <mass
+        value="1.28473302906848" />
+      <inertia
+        ixx="0.0309407894006289"
+        ixy="4.30543208060378E-05"
+        ixz="3.82039295580686E-06"
+        iyy="0.0552002635176191"
+        iyz="6.56450968178348E-05"
+        izz="0.0309385494659594" />
+    </inertial>
+    <visual>
+      <origin
+        xyz="0 0 0"
+        rpy="0 0 0" />
+      <geometry>
+        <mesh
+          filename="package://quad_simulator/meshes/base_combined.STL" />
+      </geometry>
+      <material
+        name="">
+        <color
+          rgba="0.792156862745098 0.819607843137255 0.933333333333333 1" />
+      </material>
+    </visual>
+    <collision>
+      <origin
+        xyz="0 0 0"
+        rpy="0 0 0" />
+      <geometry>
+        <mesh
+          filename="package://quad_simulator/meshes/base_combined.STL" />
+      </geometry>
+    </collision>
+  </link>
     <!-- Sonar height sensor
     <xacro:sonar_sensor name="sonar" parent="base_link" ros_topic="sonar_height" update_rate="10" min_range="0.03" max_range="3.0" field_of_view="${40*pi/180}" ray_count="3">
